File: TO220-DISCRETE/TO220-DISCRETE.kicad_pcb (KiCad board)
At the start: 2 copper layers, 74.2 x 60 mm, 44 parts, among them J1 OUT, J2 VCC, J3 VEE, J4 IN, J5 GND, Q1 BC546, Q2 BC546, Q3 BC546, Q4 BD140, Q5 BD139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

Commit message: board designed
Parts:
- moved C7 84.5 mm to (144.0, 103.6)
- moved C6 64.6 mm to (119.6, 92.7), turned to 180 degrees
- moved Q3 59.7 mm to (113.5, 101.9)
- moved R16 59.7 mm to (155.5, 108.2)
- moved R15 59.7 mm to (155.5, 111.5)
- moved Q9 59.1 mm to (148.6, 95.2)
- moved R10 58.7 mm to (131.3, 112.0), turned to 180 degrees
- moved C3 58.2 mm to (131.8, 101.7)
- moved R4 58.2 mm to (159.8, 103.1)
- moved R5 57.4 mm to (149.6, 100.1)
- moved R9 50.0 mm to (121.2, 109.0), turned to 0 degrees
- moved C5 49.3 mm to (138.2, 107.7)
- moved RV1 29.9 mm to (123.2, 102.5)
- moved R7 24.5 mm to (108.5, 112.0), turned to 0 degrees
- moved Q6 18.1 mm to (123.2, 95.6)
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Routing:
- net Net-(Q1-E): track 8.66 -> 82.5 mm
- net Net-(Q6-B): track 0.00 -> 45.3 mm
- net Net-(C5-Pad1): track 53.8 -> 97.4 mm
- net Net-(Q9-B): track 0.00 -> 39.7 mm
- net Net-(Q4-C): track 18.5 -> 47.7 mm
- net Net-(D1-K): track 66.0 -> 92.7 mm
- net Net-(Q6-C): track 12.4 -> 34.1 mm
- net Net-(C3-Pad2): track 0.00 -> 19.4 mm
- net Net-(Q3-E): track 0.00 -> 11.2 mm
- net Net-(C5-Pad2): track 0.00 -> 10.5 mm
- net Net-(Q1-C): track 51.6 -> 42.0 mm
- net Net-(Q6-E): track 14.8 -> 24.2 mm
- net Net-(C7-Pad1): track 0.00 -> 8.98 mm
- net Net-(Q2-B): track 0.00 -> 8.95 mm
- net Net-(D1-A): track 4.80 -> 13.5 mm
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Other:
- board size 74.2 x 60 mm -> 80 x 55 mm
- board text added: "GND"
- board text added: "IN"
- board text removed: "GND IN"

Commit message: tweaks
Parts:
- moved G*** 1.78 mm to (116.8, 82.5)
Routing:
- net Net-(Q4-C): track 47.7 -> 50.4 mm
- net Net-(Q6-C): track 34.1 -> 36.2 mm
- net Net-(Q3-E): track 11.2 -> 13.1 mm
- net Net-(Q9-B): track 39.7 -> 40.9 mm
- net Net-(Q1-C): track 42.0 -> 43.1 mm
- net Net-(Q6-B): track 45.3 -> 46.3 mm
- net Net-(D1-K): track 92.7 -> 91.7 mm
